File: Data_Input_Output.sch (KiCad schematic (older format))
At the start: 16 parts

Commit message: updated SD card, changed mosfets
Parts:
- added C19: .1uF, symbol C
- added C20: 10uF, symbol C
- added U? (x3): Si5468DC, MODULE, symbol Si5468DC
- gave numbers to parts that had none: 16
Connections:
- net labels added: SD_CD, SD_CS, SD_MISO, SD_MOSI, SD_SCK
- wire segments 129 -> 91
- no-connect marks 1 -> 3

Commit message: Schematics updated/components generated/PCB started
Parts:
- removed U14, U15, U16: DMN3030LFG-7, MODULE, symbol DMN3030LFG-7
- added D5, D6: FM5819-W, Diodes_SMD:SMA_Standard, symbol FM5819-W
- added K1, K2: G5LE_1A4_DC3, SPEX_Parts:G5LE-1A4-DC3, symbol G5LE_1A4_DC3
- added Q1, Q2: 2N7002K, TO_SOT_Packages_SMD:SOT-23, symbol 2N7002K
- added Q3: BSS215PH6327, TO_SOT_Packages_SMD:SOT-23, symbol BSS215PH6327
- added R29, R34, R38: 10K, Resistors_SMD:R_0603, symbol R
- C17, C18, C19, C20: footprint (none) -> Capacitors_SMD:C_0603
- Q4, Q5, Q6: renamed from U?; footprint MODULE -> SPEX_Parts:ChipFet-8
- R28: footprint (none) -> Resistors_SMD:R_0603
- R30: renamed from R29; footprint (none) -> Resistors_SMD:R_0603
- R31: renamed from R30; footprint (none) -> Resistors_SMD:R_0603
- R32: renamed from R31; footprint (none) -> Resistors_SMD:R_0603
- R33: renamed from R32; footprint (none) -> Resistors_SMD:R_0603
- R35: renamed from R33; footprint (none) -> Resistors_SMD:R_0603
- R36: renamed from R34; footprint (none) -> Resistors_SMD:R_0603
- R37: renamed from R35; footprint (none) -> Resistors_SMD:R_0603
- U11: footprint SO-8 -> Power_Integrations:SO-8
- U12: footprint MODULE -> Power_Integrations:SO-8
- U13: footprint MODULE -> SPEX_Parts:SCHA4B0400
Connections:
- net labels added: Battery_In, Battery_Out, Relay_1, Relay_2, SD_PWRCTRL, User_In, User_Out
- wire segments 91 -> 131
Other:
- moved on the sheet: C17, C18, C19, C20, Q4, Q5, Q6, R28, R30, R31, R32, R33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

Commit message: updated schematic, added headers
Parts:
- added P10, P11, P12, P7, P8, P9: CONN_01X02, Connectors_JST:JST_PH_B2B-PH-K_02x2.00mm_Straight, symbol CONN_01X02
- added P3, P4, P5, P6: CONN_01X04, Connectors_JST:JST_PH_B4B-PH-K_04x2.00mm_Straight, symbol CONN_01X04
Connections:
- net +3V3: now also P3.1 (P1), P4.1 (P1), P5.1 (P1), P6.1 (P1), P7.2 (P2)
- net 3.3V_MOS_OUT: now also P7.1 (P1)
- net 5V_MOS_OUT: now also P8.1 (P1)
- net Battery_Out: now also P10.1 (P1)
- net CANH_out: now also P6.2 (P2)
- net CANL_out: now also P6.3 (P3)
- net GND: now also P10.2 (P2), P11.2 (P2), P12.2 (P2), P3.4 (P4), P4.4 (P4), P5.4 (P4), P6.4 (P4)
- net RS485_A: now also P5.3 (P3)
- net RS485_B: now also P5.2 (P2)
- net User_In: now also P11.1 (P1)
- net User_Out: now also P12.1 (P1)
- net Vbus_MOS_OUT: now also P9.1 (P1)
- new net +5V: P8.2 (P2)
- new net UART_RX_out: P4.3 (P3)
- new net UART_TX_out: P4.2 (P2)
- new net Vbus_OUT: P9.2 (P2)
- new net i2c_SCL_out: P3.3 (P3)
- new net i2c_SDA_out: P3.2 (P2)

Commit message: board layout 95% complete
Parts:
- U13: footprint SPEX_Parts:SCHA4B0400 -> SPEX_Parts:SCH4B0419
Other:
- moved on the sheet: P10, P11, P12, P3, P4, P5, P6, P7, P8, P9
