File: Data_Input_Output.sch (KiCad schematic (older format))
At the start: 26 parts, among them P3 CONN_01X04, P4 CONN_01X04, P5 CONN_01X04, P6 CONN_01X04, P7 CONN_01X02, P8 CONN_01X02, P9 CONN_01X02, Q3 BSS215PH6327, Q4 Si5468DC, Q5 Si5468DC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

Commit message: Continued tweaks, updated BOM again
Parts:
- R21, R22: value 50K -> 51K
Changed lines of the file:
@@
 P 5950 1750
 F 0 "R21" V 6030 1750 50  0000 C CNN
-F 1 "50K" V 5950 1750 50  0000 C CNN
+F 1 "51K" V 5950 1750 50  0000 C CNN
 F 2 "Resistors_SMD:R_0603" V 5880 1750 50  0001 C CNN
 F 3 "" H 5950 1750 50  0000 C CNN
@@
 P 5950 2450
 F 0 "R22" V 5850 2450 50  0000 C CNN
-F 1 "50K" V 5950 2450 50  0000 C CNN
+F 1 "51K" V 5950 2450 50  0000 C CNN
 F 2 "Resistors_SMD:R_0603" V 5880 2450 50  0001 C CNN
 F 3 "" H 5950 2450 50  0000 C CNN
