File: Spex-Mainboard-Hardware.kicad_pcb (KiCad board)
At the start: 4 copper layers, 100 x 80 mm, 129 parts, among them K1 G5LE_1A4_DC3, K2 G5LE_1A4_DC3, P1 USB_OTG, P10 CONN_01X02, P11 CONN_01X02, P12 CONN_01X02, P2 SWD Header, P3 CONN_01X04, P4 CONN_01X04, P5 CONN_01X04, P6 CONN_01X04, P7 CONN_01X02, P8 CONN_01X02, P9 CONN_01X02, Q1 2N7002K, Q101 MOS_N_numbered, Q104 MOS_N_numbered, Q105 Si3407DV, Q106 Q_PNP_BEC, Q2 2N7002K, Q3 BSS215PH6327, Q4 Si5468DC, Q5 Si5468DC, Q6 Si5468DC, SW1 SW_PUSH, U1 MKL04Z32VLC4, U10 LM4030, U105 TPS563200, U108 TPS563200, U11 MCP2551-I/SN, U12 ST1480ABDR, U13 SCHA4B0419, U14 AT45DB641E, U2 NUP2201MR6, U3 MK20DX256VLH7, U4 NUP2201MR6, U5 NUP2201MR6, U6 MMQA6V2T1G, U7 MCP9808T, U8 BME280, U9 LSM9DS1, Y1 Crystal

Commit message: updated board
Routing:
- net VBatt: track 36.6 -> 55.2 mm
- net +3V3: track 129.7 -> 136.7 mm
Changed lines of the file:
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@@
-(kicad_pcb (version 4) (host pcbnew "(2016-03-30 BZR 6657, Git fe53ec8)-product")
+(kicad_pcb (version 4) (host pcbnew 4.0.2-stable)
   (general
     (links 339)
-    (no_connects 96)
-    (area 61.191199 50.64563 184.6705 130.885001)
+    (no_connects 24)
+    (area 61.191199 50.49938 184.553 130.885001)
     (thickness 1.6)
     (drawings 4)
-    (tracks 1199)
+    (tracks 1212)
     (zones 0)
     (modules 129)
@@
   (layers
     (0 F.Cu signal)
-    (1 In1.Cu power)
-    (2 In2.Cu power hide)
-    (31 B.Cu mixed)
+    (1 In1.Cu power hide)
+    (2 In2.Cu power)
+    (31 B.Cu mixed hide)
     (32 B.Adhes user)
     (33 F.Adhes user)
@@
   )
   (setup
-    (last_trace_width 1)
+    (last_trace_width 0.25)
     (user_trace_width 0.5)
     (user_trace_width 1)
@@
       (hpglpenspeed 20)
       (hpglpendiameter 15)
+      (hpglpenoverlay 2)
       (psnegative false)
       (psa4output false)
@@
   (segment (start 162.5346 78.994) (end 162.56 78.9686) (width 0.25) (layer In2.Cu) (net 0))
   (segment (start 105.2322 51.7144) (end 105.2322 51.7398) (width 0.25) (layer B.Cu) (net 0))
+  (segment (start 134.5 102.5) (end 135.5 103.5) (width 1) (layer In2.Cu) (net 1))
+  (segment (start 135.5 103.5) (end 135.5 102.5) (width 1) (layer In2.Cu) (net 1))
+  (segment (start 135.5 102.5) (end 135.5 99.7802) (width 1) (layer In2.Cu) (net 1))
+  (segment (start 135.4836 99.7966) (end 135.4328 99.7966) (width 0.25) (layer In2.Cu) (net 1))
+  (segment (start 135.5 99.7802) (end 135.4836 99.7966) (width 0.25) (layer In2.Cu) (net 1))
+  (segment (start 134.5 102.5) (end 134.5 99.8404) (width 1) (layer In2.Cu) (net 1))
+  (segment (start 134.5 99.8404) (end 134.5438 99.7966) (width 0.25) (layer In2.Cu) (net 1))
   (segment (start 131.5 103.5) (end 132.5 103.5) (width 0.5) (layer B.Cu) (net 1))
   (via (at 132.5 103.5) (size 0.508) (drill 0.381) (layers F.Cu B.Cu) (net 1))
@@
   (segment (start 135.5 102.5) (end 134.5 102.5) (width 0.5) (layer B.Cu) (net 1))
   (via (at 134.5 102.5) (size 0.508) (drill 0.381) (layers F.Cu B.Cu) (net 1))
-  (segment (start 135.5 103.5) (end 135.5 102.5) (width 0.5) (layer F.Cu) (net 1))
   (via (at 135.5 102.5) (size 0.508) (drill 0.381) (layers F.Cu B.Cu) (net 1))
   (segment (start 136.5 103.5) (end 135.5 103.5) (width 0.5) (layer B.Cu) (net 1))
@@
   (segment (start 169.6473 80.0093) (end 169.8625 79.7941) (width 0.25) (layer F.Cu) (net 22))
   (segment (start 166.827201 86.969601) (end 167.0812 87.2236) (width 0.25) (layer In1.Cu) (net 24))
-  (segment (start 144.672011 64.814411) (end 166.827201 86.969601) (width 0.25) (layer In1.Cu) (net 24))
-  (segment (start 112.126619 64.814411) (end 144.672011 64.814411) (width 0.25) (layer In1.Cu) (net 24))
-  (segment (start 111.91703 65.024) (end 112.126619 64.814411) (width 0.25) (layer In1.Cu) (net 24))
+  (segment (start 144.824411 64.966811) (end 166.827201 86.969601) (width 0.25) (layer In1.Cu) (net 24))
+  (segment (start 111.974219 64.966811) (end 144.824411 64.966811) (width 0.25) (layer In1.Cu) (net 24))
+  (segment (start 111.91703 65.024) (end 111.974219 64.966811) (width 0.25) (layer In1.Cu) (net 24))
   (segment (start 111.55782 65.024) (end 111.91703 65.024) (width 0.25) (layer In1.Cu) (net 24))
   (segment (start 167.0812 87.2236) (end 168.7075 87.2236) (width 0.25) (layer F.Cu) (net 24))
@@
   (segment (start 151.4236 76.0904) (end 157.5564 76.0904) (width 1.25) (layer In2.Cu) (net 77))
   (segment (start 157.5564 76.0904) (end 177.478 96.012) (width 1.25) (layer In2.Cu) (net 77))
+  (segment (start 143.5 98.5) (end 141.5 98.5) (width 1.5) (layer F.Cu) (net 78))
+  (segment (start 145.5 98.5) (end 143.5 98.5) (width 1.5) (layer F.Cu) (net 78))
+  (segment (start 147.5 100.5) (end 147.5 102.5) (width 1.5) (layer F.Cu) (net 78))
+  (segment (start 146.5 98.5) (end 147.5 99.5) (width 1.5) (layer F.Cu) (net 78))
+  (segment (start 147.5 99.5) (end 147.5 100.5) (width 1) (layer In2.Cu) (net 78))
+  (segment (start 147.5 100.5) (end 147.5 101.5) (width 1) (layer In2.Cu) (net 78))
+  (segment (start 157.4094 104.6126) (end 157.4094 104.552) (width 0.25) (layer In2.Cu) (net 78))
+  (segment (start 157.4094 104.552) (end 153.3574 100.5) (width 1) (layer In2.Cu) (net 78))
+  (segment (start 153.3574 100.5) (end 147.5 100.5) (width 1) (layer In2.Cu) (net 78))
   (segment (start 143.5 98.5) (end 143.5 100.8) (width 2) (layer F.Cu) (net 78))
   (segment (start 147.5 100.5) (end 143.8 100.5) (width 2) (layer F.Cu) (net 78))
@@
   (segment (start 147.5 100.5) (end 147.5 101.5) (width 0.5) (layer B.Cu) (net 78))
   (via (at 147.5 101.5) (size 0.508) (drill 0.381) (layers F.Cu B.Cu) (net 78))
-  (segment (start 147.5 99.5) (end 147.5 100.5) (width 0.5) (layer F.Cu) (net 78))
   (via (at 147.5 100.5) (size 0.508) (drill 0.381) (layers F.Cu B.Cu) (net 78))
-  (segment (start 146.5 98.5) (end 147.5 99.5) (width 0.5) (layer B.Cu) (net 78))
   (via (at 147.5 99.5) (size 0.508) (drill 0.381) (layers F.Cu B.Cu) (net 78))
   (segment (start 145.5 98.5) (end 146.5 98.5) (width 0.5) (layer F.Cu) (net 78))
@@
   (segment (start 139.5 98.5) (end 140.5 98.5) (width 0.5) (layer B.Cu) (net 78))
   (via (at 140.5 98.5) (size 0.508) (drill 0.381) (layers F.Cu B.Cu) (net 78))
-  (segment (start 139.5 99.5) (end 139.5 98.5) (width 0.5) (layer F.Cu) (net 78))
+  (segment (start 139.5 99.5) (end 139.5 98.5) (width 1.5) (layer F.Cu) (net 78))
   (via (at 139.5 98.5) (size 0.508) (drill 0.381) (layers F.Cu B.Cu) (net 78))
   (segment (start 139.5 100.5) (end 139.5 99.5) (width 0.5) (layer B.Cu) (net 78))
@@
     (min_thickness 0.254)
     (keepout (tracks allowed) (vias allowed) (copperpour not_allowed))
-    (fill yes (arc_segments 16) (thermal_gap 0.508) (thermal_bridge_width 0.508))
+    (fill (arc_segments 16) (thermal_gap 0.508) (thermal_bridge_width 0.508))
     (polygon
       (pts
@@
     (min_thickness 0.254)
     (keepout (tracks allowed) (vias allowed) (copperpour not_allowed))
-    (fill yes (arc_segments 16) (thermal_gap 0.508) (thermal_bridge_width 0.508))
+    (fill (arc_segments 16) (thermal_gap 0.508) (thermal_bridge_width 0.508))
     (polygon
       (pts
-        (xy 140 109) (xy 131 115) (xy 118 115) (xy 118 102.5) (xy 118 101.5)
-        (xy 118.5 101.5) (xy 140 101.5) (xy 140 109)
+        (xy 140 109) (xy 130.302 115.4938) (xy 117.983 115.4684) (xy 118 102.5) (xy 118 101.5)
+        (xy 140 101.5) (xy 140 109)
       )
     )
     (polygon
-      (pts        (xy 131 113.5) (xy 139 108) (xy 139 103) (xy 119 103) (xy 119 113.5)
-        (xy 131 113.5)
+      (pts        (xy 119 103) (xy 118.9736 114.1984) (xy 130.0226 114.1984) (xy 139 108) (xy 139 103)
+        (xy 119 103)
       )
     )

Commit message: board layout 95% complete
Parts:
- added R18: 10K, Resistors_SMD:R_0603, F.Cu at (115.6, 64.3)
- U13: footprint SPEX_Parts:SCHA4B0400 -> SPEX_Parts:SCH4B0419
- moved U13 20.9 mm to (99.9, 65.4), turned to 90 degrees
- moved Y1 1.47 mm to (117.9, 81.0)
- moved R35 0.18 mm to (168.8, 73.4)
- moved Q4 0.18 mm to (172.7, 72.4)
Connections:
- C114 pad 2: /Power Distribution/VBus -> Vbus
- C118 pad 2: /Power Distribution/VBus -> Vbus
- C120 pad 1: /Power Distribution/VBus -> Vbus
- P2 pad 10: (no net) -> RESET_b
- P2 pad 6: (no net) -> Net-(P2-Pad6)
- P2 pad 7: (no net) -> Net-(P2-Pad7)
- P2 pad 8: (no net) -> Net-(P2-Pad8)
- P2 pad 9: (no net) -> Net-(P2-Pad9)
- P9 pad 2: (no net) -> Vbus
- Q101 pad 1: /Power Distribution/VBus -> Vbus
- Q104 pad 1: /Power Distribution/VBus -> Vbus
- Q105 pad 1: /Power Distribution/VBus -> Vbus
- Q105 pad 2: /Power Distribution/VBus -> Vbus
- Q105 pad 5: /Power Distribution/VBus -> Vbus
- Q105 pad 6: /Power Distribution/VBus -> Vbus
- Q3 pad 3: (no net) -> Net-(Q3-Pad3)
- R126 pad 2: /Power Distribution/VBus -> Vbus
- R130 pad 1: /Power Distribution/VBus -> Vbus
- R140 pad 2: /Power Distribution/VBus -> Vbus
- R141 pad 1: /Power Distribution/VBus -> Vbus
- U1 pad 1: (no net) -> Net-(U1-Pad1)
- U1 pad 11: (no net) -> Net-(U1-Pad11)
- U1 pad 12: (no net) -> Net-(U1-Pad12)
- U1 pad 13: (no net) -> Net-(U1-Pad13)
- U1 pad 14: (no net) -> Net-(U1-Pad14)
- U1 pad 19: (no net) -> Net-(U1-Pad19)
- U1 pad 2: (no net) -> Net-(U1-Pad2)
- U1 pad 20: (no net) -> Net-(U1-Pad20)
- U1 pad 21: (no net) -> Net-(U1-Pad21)
- U1 pad 22: (no net) -> Net-(U1-Pad22)
- U1 pad 23: (no net) -> Net-(U1-Pad23)
- U1 pad 24: (no net) -> Net-(U1-Pad24)
- U1 pad 25: (no net) -> RESET_b
- U1 pad 26: (no net) -> Net-(U1-Pad26)
- U1 pad 27: (no net) -> Net-(U1-Pad27)
- U1 pad 28: (no net) -> Net-(U1-Pad28)
- U1 pad 29: (no net) -> Net-(U1-Pad29)
- U1 pad 30: (no net) -> Net-(U1-Pad30)
- U1 pad 31: (no net) -> Net-(U1-Pad31)
- U1 pad 32: (no net) -> Net-(U1-Pad32)
- U1 pad 7: (no net) -> Net-(U1-Pad7)
- U1 pad 8: /PTA4 -> RESET_b
- U1 pad 9: (no net) -> Net-(U1-Pad9)
- U10 pad 1: (no net) -> Net-(U10-Pad1)
- U10 pad 3: (no net) -> Net-(U10-Pad3)
- U105 pad 3: /Power Distribution/VBus -> Vbus
- U108 pad 3: /Power Distribution/VBus -> Vbus
- U11 pad 5: (no net) -> Net-(U11-Pad5)
- U14 pad 3: (no net) -> Flash_Reset
- U14 pad 5: (no net) -> +3V3
- U2 pad 3: (no net) -> Net-(U2-Pad3)
- U2 pad 4: (no net) -> Net-(U2-Pad4)
- U3 pad 12: (no net) -> Net-(U3-Pad12)
- U3 pad 18: (no net) -> Net-(U3-Pad18)
- U3 pad 19: (no net) -> Net-(U3-Pad19)
- U3 pad 20: (no net) -> Net-(U3-Pad20)
- U3 pad 26: (no net) -> Net-(U3-Pad26)
- U3 pad 27: (no net) -> Net-(U3-Pad27)
- U3 pad 34: /PTA4 -> RESET_b
- U3 pad 42: (no net) -> Net-(U3-Pad42)
- U3 pad 43: (no net) -> Flash_Reset
- U3 pad 45: (no net) -> SD_Detect
- U3 pad 61: (no net) -> Net-(U3-Pad61)
- U3 pad 62: (no net) -> Net-(U3-Pad62)
- U3 pad 63: (no net) -> Net-(U3-Pad63)
- U3 pad 64: (no net) -> Net-(U3-Pad64)
- U3 pad 8: (no net) -> Net-(U3-Pad8)
- U4 pad 3: (no net) -> Net-(U4-Pad3)
- U4 pad 4: (no net) -> Net-(U4-Pad4)
- U5 pad 3: (no net) -> Net-(U5-Pad3)
- U5 pad 4: (no net) -> Net-(U5-Pad4)
- U7 pad 3: (no net) -> /HAB Sensors/TempAlert
- U9 pad 10: (no net) -> Net-(U9-Pad10)
- U9 pad 11: (no net) -> Net-(U9-Pad11)
- U9 pad 12: (no net) -> Net-(U9-Pad12)
- U9 pad 13: (no net) -> Net-(U9-Pad13)
- U9 pad 9: (no net) -> Net-(U9-Pad9)
Routing:
- net Vbus: track 0.00 -> 161.3 mm, vias 0 -> 24
- net /Power Distribution/VBus: track 103.7 -> 0.00 mm, vias 24 -> 0
- net +5V: track 32.1 -> 123.9 mm
- net VBatt: track 55.2 -> 115.6 mm
- net RESET_b: track 0.00 -> 47.0 mm, vias 0 -> 2
- net SD_Detect: track 0.00 -> 35.4 mm, vias 0 -> 2
- net GND: track 269.8 -> 300.8 mm, vias 46 -> 49
- net SPI0_CS0: track 5.10 -> 30.4 mm, vias 1 -> 2
- net SPI0_MOSI: track 15.4 -> 34.1 mm, vias 2 -> 3
- net SPI0_SCK: track 11.7 -> 30.0 mm, vias 0 -> 2
- net SPI0_MISO: track 21.5 -> 37.2 mm, vias 0 -> 2
- net /PTA4: track 12.8 -> 0.00 mm
- net Flash_Reset: track 0.00 -> 11.5 mm, vias 0 -> 2
- net Net-(U3-Pad32): track 0.00 -> 7.99 mm, vias 0 -> 2
- net /Data_Input_Output/3.3V_MOS_OUT: track 0.00 -> 7.03 mm
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- added copper zone on F.Cu, net /Data_Input_Output/3.3V_MOS_OUT
- added copper zone on F.Cu, net /Data_Input_Output/Vbus_MOS_OUT
Other:
- board text added: "RIT SPEX HAB 2 MAINBOARD DESIGNERS: MATTHEW GLAZER CHRIS CULPEPPER"
- board text added: "Revision: 1 Design Date: 4/16"
- board text added: "TIGRIS AD ASTRA"
