File: Spex-Mainboard-Hardware.sch (KiCad schematic (older format))
At the start: 36 parts, among them P1 USB_OTG, P2 SWD Header, SW1 SW_PUSH, U1 MKL04Z32VLC4, U14 AT45DB641E, U2 NUP2201MR6, U3 MK20DX256VLH7, U4 NUP2201MR6, U5 NUP2201MR6, U6 MMQA6V2T1G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

Commit message: completed first revision of the board.
Connections:
- wire segments 249 -> 218
Changed lines of the file:
@@
 $EndComp
 Wire Wire Line
-	1350 900  1600 900
-Wire Wire Line
-	1600 900  1850 900
-Wire Wire Line
-	1850 900  2100 900
+	1350 900  2100 900
 Connection ~ 1850 900
 Wire Wire Line
@@
 	7500 5300 7250 5300
 Wire Wire Line
-	7250 5300 7250 5400
-Wire Wire Line
-	7250 5400 7250 5850
+	7250 5300 7250 5850
 Wire Wire Line
 	7500 5400 7250 5400
@@
 	5300 4500 5800 4500
 Wire Wire Line
-	2200 2500 2500 2500
-Wire Wire Line
-	2500 2500 2800 2500
+	2200 2500 2800 2500
 Wire Wire Line
 	9550 1550 9650 1550
@@
 	9050 2350 11050 2350
 Wire Wire Line
-	11050 2100 11050 2350
-Wire Wire Line
-	11050 2350 11050 2400
+	11050 2100 11050 2400
 Connection ~ 11050 2350
 Wire Wire Line
@@
 	8000 1450 8000 1550
 Wire Wire Line
-	7750 1950 7750 2050
-Wire Wire Line
-	7750 2050 7750 2150
-Wire Wire Line
-	7500 2050 7750 2050
-Wire Wire Line
-	7750 2050 8000 2050
+	7750 1950 7750 2150
+Wire Wire Line
+	7500 2050 8000 2050
 Wire Wire Line
 	8000 2050 8000 1950
@@
 	3100 6550 2950 6550
 Wire Wire Line
-	3100 1300 4400 1300
-Wire Wire Line
-	4400 1300 4550 1300
+	3100 1300 4550 1300
 Wire Wire Line
 	3700 1500 3700 1400
 Wire Wire Line
-	3400 1400 3700 1400
-Wire Wire Line
-	3700 1400 4550 1400
-Wire Wire Line
-	1450 3100 1950 3100
-Wire Wire Line
-	1950 3100 2050 3100
+	3400 1400 4550 1400
+Wire Wire Line
+	1450 3100 2050 3100
 Wire Wire Line
 	1450 3100 1450 3050
@@
 Connection ~ 1950 3100
 Wire Wire Line
-	1450 3400 1950 3400
-Wire Wire Line
-	1950 3400 2050 3400
+	1450 3400 2050 3400
 Wire Wire Line
 	1450 3400 1450 3450
@@
 	4550 3400 4400 3400
 Wire Wire Line
-	5750 4100 6150 4100
-Wire Wire Line
-	6150 4100 6350 4100
+	5750 4100 6350 4100
 Wire Wire Line
 	7550 4650 7450 4650
@@
 	3400 1550 3400 1400
 Wire Wire Line
-	2500 1550 2550 1550
-Wire Wire Line
-	2550 1550 3400 1550
+	2500 1550 3400 1550
 Connection ~ 3700 1400
 Wire Wire Line
 	2500 1650 2800 1650
 Wire Wire Line
-	2500 1850 3300 1850
-Wire Wire Line
-	3300 1850 3350 1850
+	2500 1850 3350 1850
 Wire Wire Line
 	3300 1750 3300 1700
 Wire Wire Line
-	2500 1750 2600 1750
-Wire Wire Line
-	2600 1750 3300 1750
+	2500 1750 3300 1750
 Wire Wire Line
 	3300 1700 3350 1700
@@
 	2100 1350 2550 1350
 Wire Wire Line
-	2550 1350 2550 1550
-Wire Wire Line
-	2550 1550 2550 2250
+	2550 1350 2550 2250
 Connection ~ 2550 1550
 Wire Wire Line
@@
 	4550 1700 4400 1700
 Wire Wire Line
-	4400 1300 4400 1700
-Wire Wire Line
-	4400 1700 4400 2300
-Wire Wire Line
-	4400 2300 4400 2400
+	4400 1300 4400 2400
 Connection ~ 4400 1300
 Wire Wire Line
-	3850 2600 4050 2600
-Wire Wire Line
-	4050 2600 4450 2600
-Wire Wire Line
-	4450 2600 4550 2600
+	3850 2600 4550 2600
 Wire Wire Line
 	3850 2600 3850 2650
@@
 Connection ~ 1600 900
 Wire Wire Line
-	1350 1200 1600 1200
-Wire Wire Line
-	1600 1200 1850 1200
-Wire Wire Line
-	1850 1200 2100 1200
+	1350 1200 2100 1200
 Connection ~ 1850 1200
 Connection ~ 1600 1200
@@
 	4050 2700 4150 2700
 Wire Wire Line
-	4050 2300 4050 2600
-Wire Wire Line
-	4050 2600 4050 2700
+	4050 2300 4050 2700
 Connection ~ 4050 2600
 Wire Wire Line
-	5750 3800 7050 3800
-Wire Wire Line
-	7050 3800 7100 3800
-Wire Wire Line
-	5750 3700 6900 3700
-Wire Wire Line
-	6900 3700 7100 3700
+	5750 3800 7100 3800
+Wire Wire Line
+	5750 3700 7100 3700
 Wire Wire Line
 	6250 3500 5750 3500
@@
 	5750 2300 6300 2300
 Wire Wire Line
-	3950 1100 4150 1100
-Wire Wire Line
-	4150 1100 4550 1100
-Wire Wire Line
-	3950 1200 4300 1200
-Wire Wire Line
-	4300 1200 4550 1200
+	3950 1100 4550 1100
+Wire Wire Line
+	3950 1200 4550 1200
 Wire Wire Line
 	3100 1250 3100 1300
@@
 	5750 1600 6300 1600
 Wire Wire Line
-	4350 2300 4400 2300
-Wire Wire Line
-	4400 2300 4550 2300
+	4350 2300 4550 2300
 Connection ~ 4400 1700
 Connection ~ 4400 2300
@@
 	6400 5800 5700 5800
 Wire Wire Line
-	6400 5450 6400 5500
-Wire Wire Line
-	6400 5500 6400 5800
-Wire Wire Line
-	6400 5800 6400 5900
+	6400 5450 6400 5900
 $Comp
 L +3.3V #PWR033
@@
 Flash_Reset
 Wire Wire Line
-	4650 5800 4850 5800
-Wire Wire Line
-	4850 5800 4900 5800
+	4650 5800 4900 5800
 Wire Wire Line
 	6300 3200 5750 3200

Commit message: updated passive values
Parts:
- C21: value C -> 1uF
Changed lines of the file:
@@
 P 6700 5750
 F 0 "C21" H 6725 5850 50  0000 L CNN
-F 1 "C" H 6725 5650 50  0000 L CNN
+F 1 "1uF" H 6725 5650 50  0000 L CNN
 F 2 "Capacitors_SMD:C_0603" H 6738 5600 50  0001 C CNN
 F 3 "" H 6700 5750 50  0000 C CNN

Commit message: creating revision 1 backup
Parts:
- Y1: symbol Crystal -> Crystal-RESCUE-Spex-Mainboard-Hardware
Changed lines of the file:
@@
 EESchema Schematic File Version 2
+LIBS:Spex-Mainboard-Hardware-rescue
 LIBS:power
 LIBS:device
@@
 LIBS:valves
 LIBS:parts
+LIBS:PRESSURE-BMP180_LGA7_
 LIBS:74xgxx
 LIBS:ac-dc
@@
 NoConn ~ 7500 5600
 $Comp
-L Crystal Y1
+L Crystal-RESCUE-Spex-Mainboard-Hardware Y1
 U 1 1 5679D91C
 P 5150 4500

Commit message: update
Parts:
- added SW2: SW_PUSH, Buttons_Switches_SMD:SW_SPST_B3S-1000, symbol SW_PUSH
Connections:
- net GND: now also SW2.2
- net SPI0_MISO: now also U3.52 (PTC7); no longer U3.51 (PTC6)
- net SPI0_MOSI: now also U3.51 (PTC6); no longer U3.52 (PTC7)
Changed lines of the file:
@@
 Text GLabel 6250 3400 2    60   Input ~ 0
 RX/TX_CTRL
+Text GLabel 6300 2400 2    60   Input ~ 0
+SPI0_MOSI
 Text GLabel 6300 2300 2    60   Input ~ 0
-SPI0_MOSI
-Text GLabel 6300 2400 2    60   Input ~ 0
 SPI0_MISO
 Text GLabel 6300 2500 2    60   Input ~ 0
@@
 Text GLabel 3100 3600 2    60   Input ~ 0
 RESET_b
+$Comp
+L SW_PUSH SW2
+U 1 1 57761B3F
+P 7900 4200
+F 0 "SW2" H 8050 4310 50  0000 C CNN
+F 1 "SW_PUSH" H 7900 4120 50  0000 C CNN
+F 2 "Buttons_Switches_SMD:SW_SPST_B3S-1000" H 7900 4200 50  0001 C CNN
+F 3 "" H 7900 4200 50  0000 C CNN
+	1    7900 4200
+	1    0    0    -1
+$EndComp
+$Comp
+L GND #PWR?
+U 1 1 57761B45
+P 8250 4300
+F 0 "#PWR?" H 8250 4050 50  0001 C CNN
+F 1 "GND" H 8250 4150 50  0000 C CNN
+F 2 "" H 8250 4300 60  0000 C CNN
+F 3 "" H 8250 4300 60  0000 C CNN
+	1    8250 4300
+	1    0    0    -1
+$EndComp
+Wire Wire Line
+	8200 4200 8250 4200
+Wire Wire Line
+	8250 4200 8250 4300
 $EndSCHEMATC

Commit message: update
Parts:
- removed SW2: SW_PUSH, Buttons_Switches_SMD:SW_SPST_B3S-1000, symbol SW_PUSH
Changed lines of the file:
@@
 $EndComp
 Wire Wire Line
-	1350 900  2100 900
+	1350 900  1600 900
+Wire Wire Line
+	1600 900  1850 900
+Wire Wire Line
+	1850 900  2100 900
 Connection ~ 1850 900
 Wire Wire Line
@@
 	7500 5300 7250 5300
 Wire Wire Line
-	7250 5300 7250 5850
+	7250 5300 7250 5400
+Wire Wire Line
+	7250 5400 7250 5850
 Wire Wire Line
 	7500 5400 7250 5400
@@
 	5300 4500 5800 4500
 Wire Wire Line
-	2200 2500 2800 2500
+	2200 2500 2500 2500
+Wire Wire Line
+	2500 2500 2800 2500
 Wire Wire Line
 	9550 1550 9650 1550
@@
 	9050 2350 11050 2350
 Wire Wire Line
-	11050 2100 11050 2400
+	11050 2100 11050 2350
+Wire Wire Line
+	11050 2350 11050 2400
 Connection ~ 11050 2350
 Wire Wire Line
@@
 	8000 1450 8000 1550
 Wire Wire Line
-	7750 1950 7750 2150
-Wire Wire Line
-	7500 2050 8000 2050
+	7750 1950 7750 2050
+Wire Wire Line
+	7750 2050 7750 2150
+Wire Wire Line
+	7500 2050 7750 2050
+Wire Wire Line
+	7750 2050 8000 2050
 Wire Wire Line
 	8000 2050 8000 1950
@@
 	3100 6550 2950 6550
 Wire Wire Line
-	3100 1300 4550 1300
+	3100 1300 4400 1300
+Wire Wire Line
+	4400 1300 4550 1300
 Wire Wire Line
 	3700 1500 3700 1400
 Wire Wire Line
-	3400 1400 4550 1400
-Wire Wire Line
-	1450 3100 2050 3100
+	3400 1400 3700 1400
+Wire Wire Line
+	3700 1400 4550 1400
+Wire Wire Line
+	1450 3100 1950 3100
+Wire Wire Line
+	1950 3100 2050 3100
 Wire Wire Line
 	1450 3100 1450 3050
@@
 Connection ~ 1950 3100
 Wire Wire Line
-	1450 3400 2050 3400
+	1450 3400 1950 3400
+Wire Wire Line
+	1950 3400 2050 3400
 Wire Wire Line
 	1450 3400 1450 3450
@@
 	3400 1550 3400 1400
 Wire Wire Line
-	2500 1550 3400 1550
+	2500 1550 2550 1550
+Wire Wire Line
+	2550 1550 3400 1550
 Connection ~ 3700 1400
 Wire Wire Line
 	2500 1650 2800 1650
 Wire Wire Line
-	2500 1850 3350 1850
+	2500 1850 3300 1850
+Wire Wire Line
+	3300 1850 3350 1850
 Wire Wire Line
 	3300 1750 3300 1700
 Wire Wire Line
-	2500 1750 3300 1750
+	2500 1750 2600 1750
+Wire Wire Line
+	2600 1750 3300 1750
 Wire Wire Line
 	3300 1700 3350 1700
@@
 	2100 1350 2550 1350
 Wire Wire Line
-	2550 1350 2550 2250
+	2550 1350 2550 1550
+Wire Wire Line
+	2550 1550 2550 2250
 Connection ~ 2550 1550
 Wire Wire Line
@@
 	4550 1700 4400 1700
 Wire Wire Line
-	4400 1300 4400 2400
+	4400 1300 4400 1700
+Wire Wire Line
+	4400 1700 4400 2300
+Wire Wire Line
+	4400 2300 4400 2400
 Connection ~ 4400 1300
 Wire Wire Line
-	3850 2600 4550 2600
+	3850 2600 4050 2600
+Wire Wire Line
+	4050 2600 4450 2600
+Wire Wire Line
+	4450 2600 4550 2600
 Wire Wire Line
 	3850 2600 3850 2650
@@
 Connection ~ 1600 900
 Wire Wire Line
-	1350 1200 2100 1200
+	1350 1200 1600 1200
+Wire Wire Line
+	1600 1200 1850 1200
+Wire Wire Line
+	1850 1200 2100 1200
 Connection ~ 1850 1200
 Connection ~ 1600 1200
@@
 	4050 2700 4150 2700
 Wire Wire Line
-	4050 2300 4050 2700
+	4050 2300 4050 2600
+Wire Wire Line
+	4050 2600 4050 2700
 Connection ~ 4050 2600
 Wire Wire Line
-	5750 3800 7100 3800
-Wire Wire Line
-	5750 3700 7100 3700
+	5750 3800 7050 3800
+Wire Wire Line
+	7050 3800 7100 3800
+Wire Wire Line
+	5750 3700 6900 3700
+Wire Wire Line
+	6900 3700 7100 3700
 Wire Wire Line
 	6250 3500 5750 3500
@@
 	5750 2300 6300 2300
 Wire Wire Line
-	3950 1100 4550 1100
-Wire Wire Line
-	3950 1200 4550 1200
+	3950 1100 4150 1100
+Wire Wire Line
+	4150 1100 4550 1100
+Wire Wire Line
+	3950 1200 4300 1200
+Wire Wire Line
+	4300 1200 4550 1200
 Wire Wire Line
 	3100 1250 3100 1300
@@
 	5750 1600 6300 1600
 Wire Wire Line
-	4350 2300 4550 2300
+	4350 2300 4400 2300
+Wire Wire Line
+	4400 2300 4550 2300
 Connection ~ 4400 1700
 Connection ~ 4400 2300
@@
 	6400 5800 5700 5800
 Wire Wire Line
-	6400 5450 6400 5900
+	6400 5450 6400 5500
+Wire Wire Line
+	6400 5500 6400 5800
+Wire Wire Line
+	6400 5800 6400 5900
 $Comp
 L +3.3V #PWR033
@@
 Flash_Reset
 Wire Wire Line
-	4650 5800 4900 5800
+	4650 5800 4850 5800
+Wire Wire Line
+	4850 5800 4900 5800
 Wire Wire Line
 	6300 3200 5750 3200
@@
 Text GLabel 3100 3600 2    60   Input ~ 0
 RESET_b
-$Comp
-L SW_PUSH SW2
-U 1 1 57761B3F
-P 7900 4200
-F 0 "SW2" H 8050 4310 50  0000 C CNN
-F 1 "SW_PUSH" H 7900 4120 50  0000 C CNN
-F 2 "Buttons_Switches_SMD:SW_SPST_B3S-1000" H 7900 4200 50  0001 C CNN
-F 3 "" H 7900 4200 50  0000 C CNN
-	1    7900 4200
-	1    0    0    -1
-$EndComp
-$Comp
-L GND #PWR?
-U 1 1 57761B45
-P 8250 4300
-F 0 "#PWR?" H 8250 4050 50  0001 C CNN
-F 1 "GND" H 8250 4150 50  0000 C CNN
-F 2 "" H 8250 4300 60  0000 C CNN
-F 3 "" H 8250 4300 60  0000 C CNN
-	1    8250 4300
-	1    0    0    -1
-$EndComp
-Wire Wire Line
-	8200 4200 8250 4200
-Wire Wire Line
-	8250 4200 8250 4300
 $EndSCHEMATC

Commit message: rev 2 of hab board in progress
Parts:
- removed U1: MKL04Z32VLC4, Housings_QFP:LQFP-32_7x7mm_Pitch0.8mm, symbol MKL04Z32VLC4
- added SW2: SW_PUSH, Buttons_Switches_SMD:SW_SPST_B3S-1000, symbol SW_PUSH
- added U1: MKL02Z32VFG4, Housings_DFN_QFN:QFN-16-1EP_3x3mm_Pitch0.5mm, symbol MKL02Z32VFG4
Connections:
- net +3V3: now also U1.1 (VDD)
- net GND: now also SW2.2, U1.2 (VSS)
- net PTA6: now also U1.6 (PTA6)
- net PTA7: now also U1.7 (PTA7)
- net PTB0: now also U1.8 (PTB0)
- net PTB1: now also U1.9 (PTB1)
- net PTB2: now also U1.10 (PTB2)
- net RESET_b: now also U1.13 (PTB5), U1.4 (PTA4)
- net Toggle: now reaches U3.64 (PTD7)
- net Toggle: now also SW2.1
Changed lines of the file:
@@
 L +3.3V #PWR026
 U 1 1 56F436CA
-P 1450 3050
-F 0 "#PWR026" H 1450 2900 50  0001 C CNN
-F 1 "+3.3V" H 1450 3190 50  0000 C CNN
-F 2 "" H 1450 3050 60  0000 C CNN
-F 3 "" H 1450 3050 60  0000 C CNN
-	1    1450 3050
+P 1650 3150
+F 0 "#PWR026" H 1650 3000 50  0001 C CNN
+F 1 "+3.3V" H 1650 3290 50  0000 C CNN
+F 2 "" H 1650 3150 60  0000 C CNN
+F 3 "" H 1650 3150 60  0000 C CNN
+	1    1650 3150
 	1    0    0    -1
 $EndComp
@@
 L GND #PWR027
 U 1 1 56F43CED
-P 1450 3450
-F 0 "#PWR027" H 1450 3200 50  0001 C CNN
-F 1 "GND" H 1450 3300 50  0000 C CNN
-F 2 "" H 1450 3450 60  0000 C CNN
-F 3 "" H 1450 3450 60  0000 C CNN
-	1    1450 3450
-	1    0    0    -1
-$EndComp
-Text HLabel 1900 4300 0    60   Input ~ 0
+P 1650 3350
+F 0 "#PWR027" H 1650 3100 50  0001 C CNN
+F 1 "GND" H 1650 3200 50  0000 C CNN
+F 2 "" H 1650 3350 60  0000 C CNN
+F 3 "" H 1650 3350 60  0000 C CNN
+	1    1650 3350
+	1    0    0    -1
+$EndComp
+Text HLabel 2100 3800 0    60   Input ~ 0
 PTA7
-Text HLabel 1900 4400 0    60   Input ~ 0
+Text HLabel 2100 3900 0    60   Input ~ 0
 PTB0
-Text HLabel 3100 4400 2    60   Input ~ 0
+Text HLabel 3300 3900 2    60   Input ~ 0
 PTB1
-Text HLabel 1900 3800 0    60   Input ~ 0
+Text HLabel 2100 3700 0    60   Input ~ 0
 PTA6
-Text HLabel 3100 4300 2    60   Input ~ 0
+Text HLabel 3300 3800 2    60   Input ~ 0
 PTB2
 Text HLabel 4400 3500 0    60   Input ~ 0
@@
 Text HLabel 7450 4650 0    60   Input ~ 0
 PTB2
-$Comp
-L MKL04Z32VLC4 U1
-U 1 1 56F588A7
-P 2500 3650
-F 0 "U1" H 2500 4400 50  0000 C CNN
-F 1 "MKL04Z32VLC4" H 2500 4500 50  0000 C CNN
-F 2 "Housings_QFP:LQFP-32_7x7mm_Pitch0.8mm" H 2650 2750 50  0001 C CNN
-F 3 "DOCUMENTATION" H 2500 2650 50  0001 C CNN
-	1    2500 3650
-	1    0    0    -1
-$EndComp
 Text HLabel 2800 1650 2    60   Input ~ 0
 PTA6
@@
 $EndComp
 Wire Wire Line
-	1350 900  1600 900
-Wire Wire Line
-	1600 900  1850 900
-Wire Wire Line
-	1850 900  2100 900
+	1350 900  2100 900
 Connection ~ 1850 900
 Wire Wire Line
@@
 	7500 5300 7250 5300
 Wire Wire Line
-	7250 5300 7250 5400
-Wire Wire Line
-	7250 5400 7250 5850
+	7250 5300 7250 5850
 Wire Wire Line
 	7500 5400 7250 5400
@@
 	5300 4500 5800 4500
 Wire Wire Line
-	2200 2500 2500 2500
-Wire Wire Line
-	2500 2500 2800 2500
+	2200 2500 2800 2500
 Wire Wire Line
 	9550 1550 9650 1550
@@
 	9050 2350 11050 2350
 Wire Wire Line
-	11050 2100 11050 2350
-Wire Wire Line
-	11050 2350 11050 2400
+	11050 2100 11050 2400
 Connection ~ 11050 2350
 Wire Wire Line
@@
 	8000 1450 8000 1550
 Wire Wire Line
-	7750 1950 7750 2050
-Wire Wire Line
-	7750 2050 7750 2150
-Wire Wire Line
-	7500 2050 7750 2050
-Wire Wire Line
-	7750 2050 8000 2050
+	7750 1950 7750 2150
+Wire Wire Line
+	7500 2050 8000 2050
 Wire Wire Line
 	8000 2050 8000 1950
@@
 	3100 6550 2950 6550
 Wire Wire Line
-	3100 1300 4400 1300
-Wire Wire Line
-	4400 1300 4550 1300
+	3100 1300 4550 1300
 Wire Wire Line
 	3700 1500 3700 1400
 Wire Wire Line
-	3400 1400 3700 1400
-Wire Wire Line
-	3700 1400 4550 1400
-Wire Wire Line
-	1450 3100 1950 3100
-Wire Wire Line
-	1950 3100 2050 3100
-Wire Wire Line
-	1450 3100 1450 3050
-Wire Wire Line
-	2050 3200 1950 3200
-Wire Wire Line
-	1950 3200 1950 3100
-Connection ~ 1950 3100
-Wire Wire Line
-	1450 3400 1950 3400
-Wire Wire Line
-	1950 3400 2050 3400
-Wire Wire Line
-	1450 3400 1450 3450
-Wire Wire Line
-	2050 3300 1950 3300
-Wire Wire Line
-	1950 3300 1950 3400
-Connection ~ 1950 3400
+	3400 1400 4550 1400
+Wire Wire Line
+	1650 3200 2250 3200
+Wire Wire Line
+	1650 3200 1650 3150
+Wire Wire Line
+	1650 3300 2250 3300
+Wire Wire Line
+	1650 3300 1650 3350
 Wire Wire Line
 	4550 3500 4400 3500
@@
 	7550 4650 7450 4650
 Wire Wire Line
-	3100 4400 2950 4400
-Wire Wire Line
-	2950 4300 3100 4300
-Wire Wire Line
-	2050 3600 1950 3600
-Wire Wire Line
-	1900 3800 2050 3800
-Wire Wire Line
-	2050 4300 1900 4300
-Wire Wire Line
-	1900 4400 2050 4400
-Wire Wire Line
-	3100 3600 2950 3600
+	3300 3900 3150 3900
+Wire Wire Line
+	3150 3800 3300 3800
+Wire Wire Line
+	2250 3500 2150 3500
+Wire Wire Line
+	2100 3700 2250 3700
+Wire Wire Line
+	2250 3800 2100 3800
+Wire Wire Line
+	2100 3900 2250 3900
+Wire Wire Line
+	3300 3500 3150 3500
 Wire Wire Line
 	3400 1550 3400 1400
 Wire Wire Line
-	2500 1550 2550 1550
-Wire Wire Line
-	2550 1550 3400 1550
+	2500 1550 3400 1550
 Connection ~ 3700 1400
 Wire Wire Line
 	2500 1650 2800 1650
 Wire Wire Line
-	2500 1850 3300 1850
-Wire Wire Line
-	3300 1850 3350 1850
+	2500 1850 3350 1850
 Wire Wire Line
 	3300 1750 3300 1700
 Wire Wire Line
-	2500 1750 2600 1750
-Wire Wire Line
-	2600 1750 3300 1750
+	2500 1750 3300 1750
 Wire Wire Line
 	3300 1700 3350 1700
@@
 	2100 1350 2550 1350
 Wire Wire Line
-	2550 1350 2550 1550
-Wire Wire Line
-	2550 1550 2550 2250
+	2550 1350 2550 2250
 Connection ~ 2550 1550
 Wire Wire Line
@@
 	4550 1700 4400 1700
 Wire Wire Line
-	4400 1300 4400 1700
-Wire Wire Line
-	4400 1700 4400 2300
-Wire Wire Line
-	4400 2300 4400 2400
+	4400 1300 4400 2400
 Connection ~ 4400 1300
 Wire Wire Line
-	3850 2600 4050 2600
-Wire Wire Line
-	4050 2600 4450 2600
-Wire Wire Line
-	4450 2600 4550 2600
+	3850 2600 4550 2600
 Wire Wire Line
 	3850 2600 3850 2650
@@
 Connection ~ 1600 900
 Wire Wire Line
-	1350 1200 1600 1200
-Wire Wire Line
-	1600 1200 1850 1200
-Wire Wire Line
-	1850 1200 2100 1200
+	1350 1200 2100 1200
 Connection ~ 1850 1200
 Connection ~ 1600 1200
@@
 	4050 2700 4150 2700
 Wire Wire Line
-	4050 2300 4050 2600
-Wire Wire Line
-	4050 2600 4050 2700
+	4050 2300 4050 2700
 Connection ~ 4050 2600
 Wire Wire Line
-	5750 3800 7050 3800
-Wire Wire Line
-	7050 3800 7100 3800
-Wire Wire Line
-	5750 3700 6900 3700
-Wire Wire Line
-	6900 3700 7100 3700
+	5750 3800 7100 3800
+Wire Wire Line
+	5750 3700 7100 3700
 Wire Wire Line
 	6250 3500 5750 3500
@@
 	5750 2300 6300 2300
 Wire Wire Line
-	3950 1100 4150 1100
-Wire Wire Line
-	4150 1100 4550 1100
-Wire Wire Line
-	3950 1200 4300 1200
-Wire Wire Line
-	4300 1200 4550 1200
+	3950 1100 4550 1100
+Wire Wire Line
+	3950 1200 4550 1200
 Wire Wire Line
 	3100 1250 3100 1300
@@
 	5750 1600 6300 1600
 Wire Wire Line
-	4350 2300 4400 2300
-Wire Wire Line
-	4400 2300 4550 2300
+	4350 2300 4550 2300
 Connection ~ 4400 1700
 Connection ~ 4400 2300
@@
 	6400 5800 5700 5800
 Wire Wire Line
-	6400 5450 6400 5500
-Wire Wire Line
-	6400 5500 6400 5800
-Wire Wire Line
-	6400 5800 6400 5900
+	6400 5450 6400 5900
 $Comp
 L +3.3V #PWR033
@@
 Flash_Reset
 Wire Wire Line
-	4650 5800 4850 5800
-Wire Wire Line
-	4850 5800 4900 5800
+	4650 5800 4900 5800
 Wire Wire Line
 	6300 3200 5750 3200
@@
 Text GLabel 8000 5600 2    60   Input ~ 0
 RESET_b
-Text GLabel 1950 3600 0    60   Input ~ 0
+Text GLabel 2150 3500 0    60   Input ~ 0
 RESET_b
-Text GLabel 3100 3600 2    60   Input ~ 0
+Text GLabel 3300 3500 2    60   Input ~ 0
 RESET_b
+$Comp
+L SW_PUSH SW2
+U 1 1 57903A7D
+P 7850 4200
+F 0 "SW2" H 8000 4310 50  0000 C CNN
+F 1 "SW_PUSH" H 7850 4120 50  0000 C CNN
+F 2 "Buttons_Switches_SMD:SW_SPST_B3S-1000" H 7850 4200 50  0001 C CNN
+F 3 "" H 7850 4200 50  0000 C CNN
+	1    7850 4200
+	1    0    0    -1
+$EndComp
+$Comp
+L GND #PWR039
+U 1 1 57903A83
+P 8200 4300
+F 0 "#PWR039" H 8200 4050 50  0001 C CNN
+F 1 "GND" H 8200 4150 50  0000 C CNN
+F 2 "" H 8200 4300 60  0000 C CNN
+F 3 "" H 8200 4300 60  0000 C CNN
+	1    8200 4300
+	1    0    0    -1
+$EndComp
+Wire Wire Line
+	8150 4200 8200 4200
+Wire Wire Line
+	8200 4200 8200 4300
+Wire Wire Line
+	7550 4200 7450 4200
+Text HLabel 6300 1100 2    60   Input ~ 0
+Toggle
+Wire Wire Line
+	6300 1100 5750 1100
+Text HLabel 7450 4200 0    60   Input ~ 0
+Toggle
+$Comp
+L MKL02Z32VFG4 U1
+U 1 1 579833B7
+P 2700 3550
+F 0 "U1" H 2700 3900 50  0000 C CNN
+F 1 "MKL02Z32VFG4" H 2700 4000 50  0000 C CNN
+F 2 "Housings_DFN_QFN:QFN-16-1EP_3x3mm_Pitch0.5mm" H 2850 2950 50  0001 C CNN
+F 3 "DOCUMENTATION" H 2700 3050 50  0001 C CNN
+	1    2700 3550
+	1    0    0    -1
+$EndComp
 $EndSCHEMATC

Commit message: the routing never ends
Connections:
- net I2C1_SCL: now also U4.1 (I/O); no longer U4.6 (I/O)
- net I2C1_SDA: now also U4.6 (I/O); no longer U4.1 (I/O)
Changed lines of the file:
@@
 	1    0    0    -1
 $EndComp
+Text GLabel 9650 900  0    60   Input ~ 0
+I2C1_SCL
 Text GLabel 10350 900  2    60   Input ~ 0
-I2C1_SCL
-Text GLabel 9650 900  0    60   Input ~ 0
 I2C1_SDA
 Text GLabel 9650 1450 0    60   Input ~ 0

Commit message: updates per week 1 meeting
Parts:
- added P14: CONN_01X02, Connect:PINHEAD1-2, symbol CONN_01X02
Connections:
- net GND: now also P14.2 (P2)
- net Toggle: now also P14.1 (P1)
- net CAN0_RX renamed I/O-2
- net CAN0_TX renamed I/O-1
