File: _autosave-Spex-Mainboard-Hardware.kicad_pcb (KiCad board)
At the start: 4 copper layers, 82 x 84.7 mm, 117 parts, among them P1 USB_OTG, P13 CONN_01X02, P14 CONN_01X02, P3 CONN_01X04, P4 CONN_01X04, P5 CONN_01X04, P6 CONN_01X04, P7 CONN_01X02, P8 CONN_01X02, P9 CONN_01X02, Q105 Si3407DV, Q106 Q_PNP_BEC, Q3 BSS215PH6327, Q4 Si5468DC, Q5 Si5468DC, Q6 Si5468DC, SW1 SW_PUSH, SW2 SW_PUSH, U1 MKL02Z32VFG4, U10 LM4030, U105 TPS563200, U108 TPS563200, U12 ST1480ABDR, U13 SCHA4B0419, U14 AT45DB641E, U2 NUP2201MR6, U3 MK20DX256VLH7, U4 NUP2201MR6, U5 NUP2201MR6, U6 MMQA6V2T1G, U7 MCP9808T, U8 BME280, U9 LSM9DS1, Y1 Crystal

Commit message: small update
getting ready to order PCB's, making sure they are good to go.
Connections:
- net VBatt renamed /Power Distribution/VBat
- P3 pad 2: I2C1_SDA -> I2C1_SCL
- P3 pad 3: I2C1_SCL -> I2C1_SDA
Routing:
- net I2C1_SCL: track 28.7 -> 57.8 mm, vias 1 -> 2
- net I2C1_SDA: track 42.8 -> 57.4 mm
- net /Power Distribution/VBat: track 0.00 -> 10.9 mm
- added copper zone on F.Cu, net VBatt
- removed copper zone on F.Cu, net /Power Distribution/VBat
Changed lines of the file:
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@@
 (kicad_pcb (version 4) (host pcbnew 4.0.2-stable)
   (general
-    (links 339)
-    (no_connects 19)
+    (links 336)
+    (no_connects 20)
     (area 112.379999 54.109999 194.480001 138.910001)
     (thickness 1.6)
     (drawings 4)
-    (tracks 1085)
+    (tracks 1096)
     (zones 0)
     (modules 117)
-    (nets 118)
+    (nets 119)
   )
   (page A4)
@@
   (net 116 I/O-1)
   (net 117 I/O-2)
+  (net 118 "/Power Distribution/VBat")
   (net_class Default "This is the default net class."
     (clearance 0.2032)
@@
     (add_net /Data_Input_Output/3.3V_MOS_OUT)
     (add_net /Data_Input_Output/5V_MOS_OUT)
-    (add_net /Data_Input_Output/Battery_Out)
     (add_net /Data_Input_Output/RS485_A)
     (add_net /Data_Input_Output/RS485_B)
-    (add_net /Data_Input_Output/User_In)
-    (add_net /Data_Input_Output/User_Out)
     (add_net /Data_Input_Output/Vbus_MOS_OUT)
     (add_net "/HAB Sensors/2.5VRefVoltage")
@@
     (add_net /PTB1)
     (add_net /PTB2)
+    (add_net "/Power Distribution/VBat")
     (add_net /Toggle)
     (add_net 3.3V_MOS_CTRL)
@@
     (add_net UART2_RX)
     (add_net UART2_TX)
-    (add_net VBatt)
     (add_net Vbus)
     (add_net Vbus_MOS_CTRL)
@@
     (fp_line (start -3.556 3.048) (end 3.556 3.048) (layer F.SilkS) (width 0.15))
     (pad 1 smd rect (at -3.7 0) (size 5.6 2.3) (layers F.Cu F.Paste F.Mask)
-      (net 23 VBatt))
+      (net 118 "/Power Distribution/VBat"))
     (pad 2 smd rect (at 3.7 0) (size 5.6 2.3) (layers F.Cu F.Paste F.Mask)
       (net 24 "Net-(D110-Pad2)"))
@@
       (net 1 +3V3))
     (pad 2 thru_hole oval (at 2 0 270) (size 1.2 1.7) (drill 0.7) (layers *.Cu *.Mask F.SilkS)
-      (net 32 I2C1_SDA))
-    (pad 3 thru_hole oval (at 4 0 270) (size 1.2 1.7) (drill 0.7) (layers *.Cu *.Mask F.SilkS)
       (net 33 I2C1_SCL))
+    (pad 3 thru_hole oval (at 4 0 270) (size 1.2 1.7) (drill 0.7) (layers *.Cu *.Mask F.SilkS)
+      (net 32 I2C1_SDA))
     (pad 4 thru_hole oval (at 6 0 270) (size 1.2 1.7) (drill 0.7) (layers *.Cu *.Mask F.SilkS)
       (net 2 GND))
@@
       (net 2 GND))
     (pad 2 thru_hole circle (at -1.75 7.91 90) (size 1.7 1.7) (drill 1.1) (layers *.Cu *.Mask F.SilkS)
-      (net 23 VBatt))
+      (net 118 "/Power Distribution/VBat"))
     (pad "" np_thru_hole circle (at 0 0 90) (size 3.5 3.5) (drill 3.1) (layers *.Cu *.Mask F.SilkS))
   )
@@
   (segment (start 131.0302 96.862) (end 138.2908 96.862) (width 0.25) (layer F.Cu) (net 31))
   (segment (start 138.2908 96.862) (end 139.0408 96.862) (width 0.25) (layer F.Cu) (net 31))
+  (segment (start 166.48 100.685) (end 177.7709 111.9759) (width 0.2032) (layer F.Cu) (net 32))
+  (segment (start 191.5048 114.0522) (end 179.8472 114.0522) (width 0.2032) (layer F.Cu) (net 32))
+  (segment (start 177.7709 111.9759) (end 177.8472 112.0522) (width 0.2032) (layer F.Cu) (net 32))
+  (segment (start 179.8472 114.0522) (end 177.7709 111.9759) (width 0.2032) (layer F.Cu) (net 32))
   (segment (start 164.605 98.135) (end 164.605 96.01) (width 0.2032) (layer F.Cu) (net 32))
   (segment (start 164.605 96.01) (end 158.805 90.21) (width 0.2032) (layer F.Cu) (net 32))
@@
   (segment (start 153.572859 90.215631) (end 155.926059 90.215631) (width 0.1524) (layer F.Cu) (net 32))
   (segment (start 155.926059 90.215631) (end 155.937859 90.227431) (width 0.1524) (layer F.Cu) (net 32))
-  (segment (start 166.48 100.685) (end 177.8472 112.0522) (width 0.2032) (layer F.Cu) (net 32))
   (segment (start 166.48 100.685) (end 164.605 98.81) (width 0.2032) (layer B.Cu) (net 32))
   (segment (start 164.605 98.81) (end 164.605 98.135) (width 0.2032) (layer B.Cu) (net 32))
   (via (at 166.48 100.685) (size 0.4572) (drill 0.3048) (layers F.Cu B.Cu) (net 32))
   (via (at 164.605 98.135) (size 0.4572) (drill 0.3048) (layers F.Cu B.Cu) (net 32))
-  (segment (start 165.605 98.06) (end 165.605 99.020566) (width 0.2032) (layer B.Cu) (net 33))
-  (segment (start 165.605 99.020566) (end 167.03 100.445566) (width 0.2032) (layer B.Cu) (net 33))
+  (segment (start 167.4241 100.6602) (end 178.8161 112.0522) (width 0.2032) (layer F.Cu) (net 33))
+  (segment (start 178.8161 112.0522) (end 191.5048 112.0522) (width 0.2032) (layer F.Cu) (net 33))
+  (segment (start 165.605 98.06) (end 165.605 98.8411) (width 0.2032) (layer B.Cu) (net 33))
+  (segment (start 165.605 98.8411) (end 167.4241 100.6602) (width 0.2032) (layer B.Cu) (net 33))
+  (via (at 167.4241 100.6602) (size 0.6) (drill 0.4) (layers F.Cu B.Cu) (net 33))
   (via (at 165.605 98.06) (size 0.4572) (drill 0.3048) (layers F.Cu B.Cu) (net 33))
   (segment (start 165.605 96.16) (end 165.605 98.06) (width 0.2032) (layer F.Cu) (net 33))
@@
   (segment (start 140.659699 100.30359) (end 140.603289 100.36) (width 0.2032) (layer B.Cu) (net 117))
   (segment (start 161.04859 100.30359) (end 140.659699 100.30359) (width 0.2032) (layer B.Cu) (net 117))
+  (segment (start 130.8608 67.9831) (end 132.6601 67.9831) (width 0.2032) (layer F.Cu) (net 118))
+  (segment (start 132.6601 67.9831) (end 133.18 67.4632) (width 0.2032) (layer F.Cu) (net 118))
+  (segment (start 133.18 67.4632) (end 133.18 66.11) (width 0.2032) (layer F.Cu) (net 118))
+  (segment (start 128.3339 70.51) (end 130.8608 67.9831) (width 0.2032) (layer F.Cu) (net 118))
+  (segment (start 124.88 70.51) (end 128.3339 70.51) (width 0.2032) (layer F.Cu) (net 118))
   (zone (net 2) (net_name GND) (layer B.Cu) (hatch edge 0.508)
     (connect_pads (clearance 0.25))
