File: power/procection.sch (KiCad schematic (older format))
At the start: 16 parts, among them Q105 Si3407DV, Q106 Q_PNP_BEC

Commit message: Added powerz
Connections:
- net at C119.1, D106.1 (K), Q105.4 (S)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: now also D110.1 (A); no longer D110.2 (K)
- net at F101.2, R152.2: now also D110.2 (K); no longer D110.1 (A)
Changed lines of the file:
@@
 F 4 "B340-13-F" H 2000 1100 60  0001 C CNN "Manufacturer PN"
 	1    2000 1100
-	1    0    0    -1
+	-1   0    0    1
 $EndComp
 $Comp

Commit message: rev 2 of hab board in progress
Parts:
- D109: footprint Transistors_SMD:sc70 -> TO_SOT_Packages_SMD:SC-70
- Q106: footprint Housings_SOT-23_SOT-143_TSOT-6:SOT-23 -> TO_SOT_Packages_SMD:SOT-23
Changed lines of the file:
@@
 F 0 "Q106" H 3750 1350 50  0000 R CNN
 F 1 "Q_PNP_BEC" H 4050 1250 50  0000 R CNN
-F 2 "Housings_SOT-23_SOT-143_TSOT-6:SOT-23" H 3650 1400 50  0001 C CNN
+F 2 "TO_SOT_Packages_SMD:SOT-23" H 3650 1400 50  0001 C CNN
 F 3 "" H 3450 1300 50  0000 C CNN
 F 4 "MMBT3906" H 3450 1300 60  0001 C CNN "Manufacturer PN"
@@
 F 0 "D109" H 5900 2100 50  0000 C CNN
 F 1 "D_Schottky_x2_Serial_AKC" H 5850 2300 50  0000 C CNN
-F 2 "Transistors_SMD:sc70" H 5850 2200 50  0001 C CNN
+F 2 "TO_SOT_Packages_SMD:SC-70" H 5850 2200 50  0001 C CNN
 F 3 "" H 5850 2200 50  0000 C CNN
 F 4 "BAV99WT1G" H 5850 2200 60  0001 C CNN "Manufacturer PN"

Commit message: continued work on power electronics
Parts:
- D110: footprint Diodes_SMD:Diode-SMA_Standard -> Diodes_SMD:SMA_Standard
Changed lines of the file:
@@
 F 0 "D110" H 2000 1200 40  0000 C CNN
 F 1 "DIODE" H 2000 1000 40  0000 C CNN
-F 2 "Diodes_SMD:Diode-SMA_Standard" H 2000 1100 60  0001 C CNN
+F 2 "Diodes_SMD:SMA_Standard" H 2000 1100 60  0001 C CNN
 F 3 "" H 2000 1100 60  0000 C CNN
 F 4 "B340-13-F" H 2000 1100 60  0001 C CNN "Manufacturer PN"
